File: sensor-board2.sch (EAGLE design)
At the start: 76 parts, among them IC1 MCP3423, IC10_ADJ LD117AS12TR, IC1_VDD=7.5V MAX4194, IC2 MPXHZ6115A6U, IC3 MPX2010, IC4 MAG3110, IC5 MMA8652FC, IC6 FXAS21002C, IC7 RFM95, IC8_5V LD117AS12TR, IC9_3.3V LD117AS12TR, IC9_3.3V1 LD117AS12TR, J2 JP7, Q1 BSS123, Q2 BSS123, X1 SMA-142-0701-801/806

Commit message: cdn
Parts:
- added D5: 1N5819, diode:1N5819
- added IC8: LM2731(X/Y), TI:LM2731(X/Y)
- added L1: POWER_INDUCTOR_SMD, micrel:POWER_INDUCTOR_SMD
Connections:
- new net N$17: D5.A, IC8.SW, L1.2
- new net N$2: IC8.VIN, L1.1
Changed lines of the file:
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@@
 <part name="R14" library="resistor" deviceset="R-EU_" device="R0805" value="2k2"/>
 <part name="GND38" library="supply1" deviceset="GND" device=""/>
+<part name="IC8" library="TI" deviceset="LM2731(X/Y)" device=""/>
+<part name="L1" library="micrel" deviceset="POWER_INDUCTOR_SMD" device=""/>
+<part name="D5" library="diode" deviceset="1N5819" device=""/>
 </parts>
 <sheets>
@@
 <instance part="R14" gate="G$1" x="53.34" y="-218.44" rot="R90"/>
 <instance part="GND38" gate="1" x="53.34" y="-226.06"/>
+<instance part="IC8" gate="G$1" x="-165.1" y="-170.18"/>
+<instance part="L1" gate="G$1" x="-162.56" y="-152.4"/>
+<instance part="D5" gate="G$1" x="-142.24" y="-167.64"/>
 </instances>
 <busses>
@@
 </segment>
 </net>
+<net name="N$2" class="0">
+<segment>
+<pinref part="IC8" gate="G$1" pin="VIN"/>
+<wire x1="-175.26" y1="-165.1" x2="-177.8" y2="-165.1" width="0.1524" layer="91"/>
+<wire x1="-177.8" y1="-165.1" x2="-177.8" y2="-152.4" width="0.1524" layer="91"/>
+<pinref part="L1" gate="G$1" pin="1"/>
+<wire x1="-177.8" y1="-152.4" x2="-167.64" y2="-152.4" width="0.1524" layer="91"/>
+</segment>
+</net>
+<net name="N$17" class="0">
+<segment>
+<pinref part="L1" gate="G$1" pin="2"/>
+<wire x1="-157.48" y1="-152.4" x2="-149.86" y2="-152.4" width="0.1524" layer="91"/>
+<wire x1="-149.86" y1="-152.4" x2="-149.86" y2="-167.64" width="0.1524" layer="91"/>
+<pinref part="IC8" gate="G$1" pin="SW"/>
+<wire x1="-149.86" y1="-167.64" x2="-152.4" y2="-167.64" width="0.1524" layer="91"/>
+<pinref part="D5" gate="G$1" pin="A"/>
+<wire x1="-149.86" y1="-167.64" x2="-144.78" y2="-167.64" width="0.1524" layer="91"/>
+<junction x="-149.86" y="-167.64"/>
+</segment>
+</net>

Commit message: cdn
Parts:
- removed L1: POWER_INDUCTOR_SMD, micrel:POWER_INDUCTOR_SMD
- added C15: 4u7/25V, rcl:CPOL-EUSMCD
- added C20: 270p, rcl:C-EUC0805
- added C21: krowka_10/25V, rcl:CPOL-EUSMCD
- added L2: POWER_INDUCTOR, miscrel:POWER_INDUCTOR
- added R15: 12k (zalecaja 13k3), resistor:R-EU_R0805
- added R16: 100k, resistor:R-EU_R0805
- added R17: 10k, resistor:R-EU_R0805
- added R18: 50k, resistor:R-EU_R0805
- Q1, Q2: value BSS123 -> AO3402; device transistor-small-signal:BSS123 -> TI:AO3402
Connections:
- new net N$19: C20.1, IC8.FB, R15.1, R16.1
- new net N$20: C15.-, C21.-, IC8.GND, R15.2
- new net N$23: C15.+, C20.2, D5.C, R16.2
- new net N$28: IC8.!SHDN!, R18.1
- net N$17: now also L2.2; no longer L1.2
- net N$2: now also C21.+, L2.1, R18.2; no longer L1.1
Other:
- note added: "R2 = R1 (Vout / 1.23 -1) R1=12k; R2=100k => Vout=11.48"
- note added: "roladowanie pojemnosci linii???"
- moved on the sheet: D5
Changed lines of the file:
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@@
 <part name="D4" library="diode" deviceset="DIODE-" device="MELF-MLL41"/>
 <part name="J2" library="jumper" deviceset="JP7" device=""/>
-<part name="Q1" library="transistor-small-signal" deviceset="BSS123" device=""/>
-<part name="Q2" library="transistor-small-signal" deviceset="BSS123" device=""/>
+<part name="Q1" library="TI" deviceset="AO3402" device=""/>
+<part name="Q2" library="TI" deviceset="AO3402" device=""/>
 <part name="R6" library="resistor" deviceset="R-EU_" device="R0805" value="4k7"/>
 <part name="R7" library="resistor" deviceset="R-EU_" device="R0805" value="10k"/>
@@
 <part name="GND38" library="supply1" deviceset="GND" device=""/>
 <part name="IC8" library="TI" deviceset="LM2731(X/Y)" device=""/>
-<part name="L1" library="micrel" deviceset="POWER_INDUCTOR_SMD" device=""/>
 <part name="D5" library="diode" deviceset="1N5819" device=""/>
+<part name="R15" library="resistor" deviceset="R-EU_" device="R0805" value="12k (zalecaja 13k3)"/>
+<part name="R16" library="resistor" deviceset="R-EU_" device="R0805" value="100k"/>
+<part name="R17" library="resistor" deviceset="R-EU_" device="R0805" value="10k"/>
+<part name="C15" library="rcl" deviceset="CPOL-EU" device="SMCD" value="4u7/25V"/>
+<part name="C20" library="rcl" deviceset="C-EU" device="C0805" value="270p"/>
+<part name="C21" library="rcl" deviceset="CPOL-EU" device="SMCD" value="krowka_10/25V"/>
+<part name="R18" library="resistor" deviceset="R-EU_" device="R0805" value="50k"/>
+<part name="L2" library="miscrel" deviceset="POWER_INDUCTOR" device=""/>
 </parts>
 <sheets>
@@
 <text x="-33.02" y="-307.34" size="1.778" layer="91">zlacze wchodzace
 na adapter - stad 5V</text>
+<text x="-165.1" y="-144.78" size="1.778" layer="91">R2 = R1 (Vout / 1.23 -1)
+R1=12k; R2=100k =&gt; Vout=11.48</text>
+<text x="165.1" y="-162.56" size="1.778" layer="91">roladowanie pojemnosci linii???</text>
 </plain>
 <instances>
@@
 <instance part="GND38" gate="1" x="53.34" y="-226.06"/>
 <instance part="IC8" gate="G$1" x="-165.1" y="-170.18"/>
-<instance part="L1" gate="G$1" x="-162.56" y="-152.4"/>
-<instance part="D5" gate="G$1" x="-142.24" y="-167.64"/>
+<instance part="D5" gate="G$1" x="-134.62" y="-167.64"/>
+<instance part="R15" gate="G$1" x="-149.86" y="-190.5" rot="R270"/>
+<instance part="R16" gate="G$1" x="-142.24" y="-172.72"/>
+<instance part="R17" gate="G$1" x="172.72" y="-177.8" rot="R90"/>
+<instance part="C15" gate="G$1" x="-132.08" y="-187.96"/>
+<instance part="C20" gate="G$1" x="-142.24" y="-182.88" rot="R90"/>
+<instance part="C21" gate="G$1" x="-190.5" y="-187.96"/>
+<instance part="R18" gate="G$1" x="-182.88" y="-170.18" rot="R180"/>
+<instance part="L2" gate="G$1" x="-162.56" y="-152.4"/>
 </instances>
 <busses>
@@
 <segment>
 <pinref part="IC8" gate="G$1" pin="VIN"/>
-<wire x1="-175.26" y1="-165.1" x2="-177.8" y2="-165.1" width="0.1524" layer="91"/>
-<wire x1="-177.8" y1="-165.1" x2="-177.8" y2="-152.4" width="0.1524" layer="91"/>
-<pinref part="L1" gate="G$1" pin="1"/>
-<wire x1="-177.8" y1="-152.4" x2="-167.64" y2="-152.4" width="0.1524" layer="91"/>
+<wire x1="-175.26" y1="-165.1" x2="-190.5" y2="-165.1" width="0.1524" layer="91"/>
+<wire x1="-190.5" y1="-165.1" x2="-190.5" y2="-152.4" width="0.1524" layer="91"/>
+<wire x1="-190.5" y1="-152.4" x2="-167.64" y2="-152.4" width="0.1524" layer="91"/>
+<pinref part="C21" gate="G$1" pin="+"/>
+<wire x1="-190.5" y1="-185.42" x2="-190.5" y2="-170.18" width="0.1524" layer="91"/>
+<junction x="-190.5" y="-165.1"/>
+<junction x="-190.5" y="-165.1"/>
+<pinref part="R18" gate="G$1" pin="2"/>
+<wire x1="-190.5" y1="-170.18" x2="-190.5" y2="-165.1" width="0.1524" layer="91"/>
+<wire x1="-187.96" y1="-170.18" x2="-190.5" y2="-170.18" width="0.1524" layer="91"/>
+<junction x="-190.5" y="-170.18"/>
+<wire x1="-190.5" y1="-165.1" x2="-195.58" y2="-165.1" width="0.1524" layer="91"/>
+<pinref part="L2" gate="G$1" pin="1"/>
 </segment>
 </net>
 <net name="N$17" class="0">
 <segment>
-<pinref part="L1" gate="G$1" pin="2"/>
 <wire x1="-157.48" y1="-152.4" x2="-149.86" y2="-152.4" width="0.1524" layer="91"/>
 <wire x1="-149.86" y1="-152.4" x2="-149.86" y2="-167.64" width="0.1524" layer="91"/>
@@
 <wire x1="-149.86" y1="-167.64" x2="-152.4" y2="-167.64" width="0.1524" layer="91"/>
 <pinref part="D5" gate="G$1" pin="A"/>
-<wire x1="-149.86" y1="-167.64" x2="-144.78" y2="-167.64" width="0.1524" layer="91"/>
+<wire x1="-149.86" y1="-167.64" x2="-137.16" y2="-167.64" width="0.1524" layer="91"/>
 <junction x="-149.86" y="-167.64"/>
-</segment>
-</net>
+<pinref part="L2" gate="G$1" pin="2"/>
+</segment>
+</net>
+<net name="N$19" class="0">
+<segment>
+<pinref part="IC8" gate="G$1" pin="FB"/>
+<pinref part="R15" gate="G$1" pin="1"/>
+<wire x1="-152.4" y1="-172.72" x2="-149.86" y2="-172.72" width="0.1524" layer="91"/>
+<wire x1="-149.86" y1="-172.72" x2="-149.86" y2="-182.88" width="0.1524" layer="91"/>
+<pinref part="R16" gate="G$1" pin="1"/>
+<wire x1="-149.86" y1="-182.88" x2="-149.86" y2="-185.42" width="0.1524" layer="91"/>
+<wire x1="-149.86" y1="-172.72" x2="-147.32" y2="-172.72" width="0.1524" layer="91"/>
+<junction x="-149.86" y="-172.72"/>
+<pinref part="C20" gate="G$1" pin="1"/>
+<wire x1="-144.78" y1="-182.88" x2="-149.86" y2="-182.88" width="0.1524" layer="91"/>
+<junction x="-149.86" y="-182.88"/>
+</segment>
+</net>
+<net name="N$20" class="0">
+<segment>
+<pinref part="R15" gate="G$1" pin="2"/>
+<pinref part="C15" gate="G$1" pin="-"/>
+<wire x1="-132.08" y1="-193.04" x2="-132.08" y2="-198.12" width="0.1524" layer="91"/>
+<wire x1="-132.08" y1="-198.12" x2="-149.86" y2="-198.12" width="0.1524" layer="91"/>
+<wire x1="-149.86" y1="-198.12" x2="-177.8" y2="-198.12" width="0.1524" layer="91"/>
+<wire x1="-177.8" y1="-198.12" x2="-177.8" y2="-175.26" width="0.1524" layer="91"/>
+<pinref part="IC8" gate="G$1" pin="GND"/>
+<wire x1="-177.8" y1="-175.26" x2="-175.26" y2="-175.26" width="0.1524" layer="91"/>
+<wire x1="-149.86" y1="-195.58" x2="-149.86" y2="-198.12" width="0.1524" layer="91"/>
+<junction x="-149.86" y="-198.12"/>
+<pinref part="C21" gate="G$1" pin="-"/>
+<wire x1="-190.5" y1="-193.04" x2="-190.5" y2="-198.12" width="0.1524" layer="91"/>
+<wire x1="-190.5" y1="-198.12" x2="-177.8" y2="-198.12" width="0.1524" layer="91"/>
+<junction x="-177.8" y="-198.12"/>
+</segment>
+</net>
+<net name="N$23" class="0">
+<segment>
+<pinref part="C20" gate="G$1" pin="2"/>
+<pinref part="C15" gate="G$1" pin="+"/>
+<wire x1="-137.16" y1="-182.88" x2="-132.08" y2="-182.88" width="0.1524" layer="91"/>
+<wire x1="-132.08" y1="-182.88" x2="-132.08" y2="-185.42" width="0.1524" layer="91"/>
+<pinref part="R16" gate="G$1" pin="2"/>
+<wire x1="-137.16" y1="-172.72" x2="-127" y2="-172.72" width="0.1524" layer="91"/>
+<wire x1="-127" y1="-172.72" x2="-127" y2="-167.64" width="0.1524" layer="91"/>
+<pinref part="D5" gate="G$1" pin="C"/>
+<wire x1="-127" y1="-167.64" x2="-132.08" y2="-167.64" width="0.1524" layer="91"/>
+<wire x1="-132.08" y1="-182.88" x2="-127" y2="-182.88" width="0.1524" layer="91"/>
+<wire x1="-127" y1="-182.88" x2="-127" y2="-172.72" width="0.1524" layer="91"/>
+<junction x="-132.08" y="-182.88"/>
+<junction x="-127" y="-172.72"/>
+</segment>
+</net>
+<net name="N$28" class="0">
+<segment>
+<pinref part="IC8" gate="G$1" pin="!SHDN!"/>
+<pinref part="R18" gate="G$1" pin="1"/>
+<wire x1="-175.26" y1="-170.18" x2="-177.8" y2="-170.18" width="0.1524" layer="91"/>
+</segment>
+</net>

Commit message: cdn
Other:
- note added: "++ zabezpieczenia antyprzepieciowe i bezpieczniki?? moze ledy wskazujace awarie"
- note added: "++ zabezpieczenia przepieciowe i wskaxniki stanu/awarii na ledach"
- note removed: "++ zabezpieczenia przepieciowe"
Changed lines of the file:
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@@
 5. doubled capacitors VREGD and VDDIO reduced to single C12 100n</text>
 <text x="55.88" y="-208.28" size="1.778" layer="97">0.1-2V output range</text>
-<text x="-88.9" y="-20.32" size="1.778" layer="91">++ zabezpieczenia przepieciowe</text>
+<text x="-88.9" y="-15.24" size="1.778" layer="91">++ zabezpieczenia przepieciowe i wskaxniki stanu/awarii na ledach</text>
 <text x="-88.9" y="-25.4" size="1.778" layer="91">++ boost -&gt;12V</text>
 <text x="-33.02" y="-307.34" size="1.778" layer="91">zlacze wchodzace
@@
 R1=12k; R2=100k =&gt; Vout=11.48</text>
 <text x="165.1" y="-162.56" size="1.778" layer="91">roladowanie pojemnosci linii???</text>
+<text x="-88.9" y="-20.32" size="1.778" layer="91">++ zabezpieczenia antyprzepieciowe i bezpieczniki?? moze ledy wskazujace awarie</text>
 </plain>
 <instances>

Commit message: IO discrete buffers
Parts:
- added IC10, IC9: (no value), TI:TL431-ASA
- added IC11: 4504D, 45xx:4504D
- added Q11, Q12, Q13, Q14, Q15, Q16, Q3, Q4, Q5, Q6, Q7, Q8, Q9: (no value), TI:AO3402
- added R19: 82k, resistor:R-EU_R0805
- added R20: 33k, resistor:R-EU_R0805
- added R21, R22, R25, R26, R30, R32, R34, R36, R38, R40: 10k, resistor:R-EU_R0805
- added R23: 2k2, resistor:R-EU_R0805
- added R24, R27, R31, R33, R35, R37, R39, R41: 4k7, resistor:R-EU_R0805
- added ZOLTY_TANTAL1: 22uF/10v, rcl:CPOL-EUSMCB
- IC1_VDD=7.5V: value MAX4194 -> (none)
- IC2: value MPXHZ6115A6U -> (none)
- IC3: value MPX2010 -> (none)
- IC4: value MAG3110 -> (none)
- IC5: value MMA8652FC -> (none)
- IC6: value FXAS21002C -> (none)
- IC7: value RFM95 -> (none)
- IC8: value LM2731(X/Y) -> (none)
- L2: value POWER_INDUCTOR -> (none)
- Q1, Q2: value AO3402 -> (none)
- R7: value 10k -> 4k7
Connections:
- removed net REF3V3: Q1.G, Q2.G, R6.1, R7.2
- new net INT1_B: JP3.2, Q12.D, R32.1
- new net INT1_XX_B: JP4.1, Q16.D, R40.1
- new net INT1_X_B: JP4.2, Q15.D, R38.1
- new net INT2_B: JP3.1, Q13.D, R34.1
- new net INT2_X_B: JP4.3, Q14.D, R36.1
- new net MISO_B: Q3.D
- new net MOSI_B: Q4.D
- new net N$21: IC9.R, R19.2, R20.1
- new net N$22: IC10.R, IC9.C, R21.1, R22.2, ZOLTY_TANTAL1.-
- new net N$24: Q11.S, R31.1
- new net N$27: IC10.A
- new net N$29: IC10.C, R26.1
- new net N$30: R20.2, R21.2, R26.2, ZOLTY_TANTAL1.+
- new net N$33: Q12.S, R33.1
- new net N$35: Q13.S, R35.1
- new net N$37: Q14.S, R37.1
- new net N$39: Q15.S, R39.1
- new net N$41: Q16.S, R41.1
- new net NSS_B: Q6.D
- new net RESET_B: Q7.D
- new net RST_B_B: JP3.3, Q11.D, R30.1
- new net SCK_B: Q5.D
- new net SCL2_B: JP2.3, Q8.D, R17.1
- new net SDA2_B: JP2.2, Q9.D, R25.1
- new net V_LOC: Q3.G, Q4.G, Q5.G, Q6.G, Q7.G, R23.1
- net +3V3: now also R23.2
- net +5V: now also Q1.G, Q2.G, R17.2, R25.2, R30.2, R32.2, R34.2, R36.2, R38.2, R40.2, R7.2
- net GND: no longer R7.1
- net INT1: no longer JP3.2
- net INT1_X: no longer JP4.2
- net INT1_XX: no longer JP4.1
- net INT2: no longer JP3.1
- net INT2_X: no longer JP4.3
- net MISO: now also Q3.S
- net MOSI: now also Q4.S; no longer J2.5
- net NSS: now also Q6.S; no longer J2.3
- net RESET: now also Q7.S; no longer J2.2
- net RST_B: no longer JP3.3
- net SCK: now also Q5.S; no longer J2.4
- net SCL-R: now also R7.1
- net SCL2: now also Q8.S, R24.1; no longer JP2.3
- net SDA-R: now also R6.1
- net SDA2: now also Q9.S, R27.1; no longer JP2.2
- net VCCIO: now also Q11.G, Q12.G, Q13.G, Q14.G, Q15.G, Q16.G, Q8.G, Q9.G, R24.2, R27.2, R31.2, R33.2, R35.2, R37.2, R39.2, R41.2
Other:
- note added: "1-100mA zakres dzialania TL431 ten uklad niech trzyma niski prad bo jedynie monitoruje napiacia"
- note added: "2V5 REF"
- note added: "3.53304 @2.52 3.46294 @2.47"
- note added: "Brak zasilania po stronie ukladu - brak napiecia na IO, ktore mogloby uszkodzic porty (Vin + 0.3V) Dodatkowo level shifter, po prawej moze byc dowolne napiecie >2.5V"
- note added: "HIGH 3.6V"
- note added: "I_REF <=1-4uA I_dzielnika=30uA"
- note added: "LOW 3V"
- note added: "po tej stronie, czyli od mastera prawdopodobnie sa pullupy"
- note added: "revision: 1. signal inputs for MCP3432 adjusted to range -2:+2V by adding voltage divider to MPXHZ6115 and adjusting gain of MPX2010 signal to G=79.1 2. protection diodes for LM stabilizers added 3. NSS -SPI selection pin- for RFM95 attached to connector 4. added logic converters 3V3<->5V for MCP3432 5. doubled capacitors VREGD and VDDIO reduced to single C12 100n 6. NMOF comm. buffers as prevent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"
- note removed: "revision: 1. signal inputs for MCP3432 adjusted to range -2:+2V by adding voltage divider to MPXHZ6115 and adjusting gain of MPX2010 signal to G=79.1 2. protection diodes for LM stabilizers added 3. NSS -SPI selection pin- for RFM95 attached to connector 4. added logic converters 3V3<->5V for MCP3432 5. doubled capacitors VREGD and VDDIO reduced to single C12 100n"
- note removed: "roladowanie pojemnosci linii???"
- moved on the sheet: IC7, JP2, JP3, JP4, PAD2, PAD3, PAD4, PAD5, PAD6, PAD7, R17, R6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

Commit message: overvoltage protection
Parts:
- removed IC10: (no value), TI:TL431-ASA
- removed IC11: 4504D, 45xx:4504D
- removed R26: 10k, resistor:R-EU_R0805
- removed ZOLTY_TANTAL1: 22uF/10v, rcl:CPOL-EUSMCB
- added C22: 330uF/6V2, rcl:CPOL-EUSMCD
- added C23: 100n, rcl:C-EUC0805
- added D6, D7: (no value), diode:DIODE-MELF-MLL41
- added IC9_3.3V2: LD117AS12TR, v-reg:LD117AS12TR
- added LED4: (no value), eagle-ltspice:LED_E
- added Q10, Q17: IRF540, transistor-power:IRF540
- added Q18: BC807-16LT1SMD, transistor-pnp:BC807-16LT1SMD
- added R28: 27k, resistor:R-EU_R0805
- added R29: 15k, resistor:R-EU_R0805
- added R42: 3k3, resistor:R-EU_R0805
- added T1: BC847, transistor:BC847
- R21: value 10k -> 1k5
- R22: value 10k -> 330k
Connections:
- new net N$26: Q17.G, Q18.C, R42.2
- new net N$31: IC9_3.3V2.ADJ
- new net N$32: C23.2
- new net N$34: IC9.C, R29.1
- new net N$38: R42.1
- new net N$42: Q10.G, Q17.D, R28.2
- net N$21: now also C23.1
- net N$22: now also IC9_3.3V2.OUT, Q10.D; no longer IC10.R, IC9.C, R21.1, R22.2, ZOLTY_TANTAL1.-
- net N$27: now also Q18.B, R22.1, R29.2; no longer IC10.A
- net N$29: now also IC9_3.3V2.IN, Q18.E, R22.2, R28.1; no longer IC10.C, R26.1
- net N$30: now also Q10.S; no longer R21.2, R26.2, ZOLTY_TANTAL1.+
Other:
- note added: "2V5 min"
- note added: "translacja 3v3 -> 3v3 3v3 <- 5 (3v3, 3v3-0,7 w najgorszym razie)"
- moved on the sheet: IC9, R19, R21, R22

Commit message: overvoltage protection fix
Parts:
- removed C23: 100n, rcl:C-EUC0805
- removed D6, D7: (no value), diode:DIODE-MELF-MLL41
- removed Q17: IRF540, transistor-power:IRF540
- removed R21: 1k5, resistor:R-EU_R0805
- removed R28: 27k, resistor:R-EU_R0805
- removed T1: BC847, transistor:BC847
- added Q19: IRLML2060, miscrel:IRLML2060
- added R26: 1k, resistor:R-EU_R0805
- IC2: value (none) -> MPXHZ6115A6U
- IC3: value (none) -> MPX2010
- IC4: value (none) -> MAG3110
- IC5: value (none) -> MMA8652FC
- IC6: value (none) -> FXAS21002C
- IC7: value (none) -> RFM95
- IC8: value (none) -> LM2731(X/Y)
- IC9: value (none) -> TLV431 (1.24VREF)
- Q10: value IRF540 -> (none); device transistor-power:IRF540 -> transistor-power:P-MOSFET-SO8
- R19: value 82k -> 100k
- R20: value 33k -> 180k
- R22: value 330k -> 1M
- R29: value 15k -> 100k
Connections:
- removed net N$26: Q17.G, Q18.C, R42.2
- removed net N$42: Q10.G, Q17.D, R28.2
- new net N$36: Q19.S
- new net N$40: Q19.D, R26.2
- new net S3V3_FAULT: Q10.G, Q18.C, Q19.G, R42.2
- net N$21: no longer C23.1
- net N$22: now also Q10.S; no longer Q10.D
- net N$27: no longer R22.1
- net N$29: now also LED4.A; no longer R28.1
- net N$30: now also Q10.D; no longer Q10.S
- net N$32: now also LED4.C, R26.1; no longer C23.2
- net N$34: now also R22.1
Other:
- note added: "3.5784 @1.278 3.472 @ typ 1.24 3.3656 @1.202 przy bledzie dzielnika .46% (rez. 1%) najwyzsze mozliwe napiecie to 3.595"
- note removed: "1-100mA zakres dzialania TL431 ten uklad niech trzyma niski prad bo jedynie monitoruje napiacia"
- note removed: "2V5 REF"
- note removed: "2V5 min"
- note removed: "3.53304 @2.52 3.46294 @2.47"
- note removed: "HIGH 3.6V"
- note removed: "I_REF <=1-4uA I_dzielnika=30uA"
- note removed: "LOW 3V"
- moved on the sheet: IC9_3.3V2, LED4, R19, R20, R29, R42

Commit message: 12/6/5 voltages added
Parts:
- removed D5: 1N5819, diode:1N5819
- removed IC9_3.3V2: LD117AS12TR, v-reg:LD117AS12TR
- removed L2: (no value), miscrel:POWER_INDUCTOR
- added C23, C24: 1u/50V, rcl:C-EUC1206
- added C25: 560p/50V, rcl:C-EUC1206
- added C26, C29: 4u7/16V, resistor:C-EUC1206
- added C28, C30: 22u/25V, rcl:CPOL-EUC/6032-28R
- added C31: 470p/50V, rcl:C-EUC1206
- added D6: 3v3, diode:ZENER-DIODESOD80C
- added D7: 1N5819, diode:1N5819
- added D8, D9: 4001, diode:DIODE-DO-214AC
- added IC10: LM2731(X/Y), TI:LM2731(X/Y)
- added IC11: TLV702, TI:TLV702
- added IC12: TC1044SEOA, TI:TC1044SEOA
- added IC13: MIC5209, TI:MIC5209
- added IC15: LM393D, linear:LM393D
- added L1: 10uH, miscrel:POWER_INDUCTOR
- added Q17: DMP3130L, miscrel:DMP3130L
- added R21, R48: 1M, resistor:R-EU_R0805
- added R28: 12k, resistor:R-EU_R0805
- added R43, R45: 47k, resistor:R-EU_R0805
- added R44, R47: 56k, resistor:R-EU_R0805
- added R46: 330k, resistor:R-EU_R0805
- added R51: 100k, resistor:R-EU_R0805
- added R52: 15k, resistor:R-EU_R0805
- C15: value 4u7/25V -> 22u/25V; device rcl:CPOL-EUSMCD -> rcl:CPOL-EUC/6032-28R
- C20: value 270p -> 22u/25V; device rcl:C-EUC0805 -> rcl:CPOL-EUC/6032-28R
- C21: value krowka_10/25V -> 470p/50V; device rcl:CPOL-EUSMCD -> rcl:C-EUC1206
- C22: value 330uF/6V2 -> 1u/50V; device rcl:CPOL-EUSMCD -> rcl:C-EUC1206
- IC8: value LM2731(X/Y) -> MIC5209; device TI:LM2731(X/Y) -> TI:MIC5209
- LED4: value (none) -> FAULT IND RED
- Q10: value (none) -> DMP3130L; device transistor-power:P-MOSFET-SO8 -> miscrel:DMP3130L
- R15: value 12k (zalecaja 13k3) -> 33k
- R18: value 50k -> 56k
Connections:
- net N$30 renamed 3V3_FOR_LORA
- removed net S3V3_FAULT: Q10.G, Q18.C, Q19.G, R42.2
- new net BOOST_SENS_A+: C31.2, IC13.ADJ, R45.1, R46.1
- new net BOOST_SENS_A-: R51.1, R52.2
- new net LOW_SHDN_6V: IC10.!SHDN!, R44.1
- new net N$26: IC11.EN
- new net N$30: D7.A, IC10.SW, L1.2
- new net N$42: IC15A.+IN
- new net N$43: C28.+, D9.C, IC13.VIN, R18.1
- new net N$44: C22.1, IC13.VO, R46.2, R51.2
- new net N$45: IC15A.-IN
- new net N$46: IC13.EN, R18.2
- new net POWER_FAULT_3V3_PLOGIC_CMOS: D6.C, R21.1
- new net PUMP_HI_TO_SHDN: Q17.G
- new net REHREH: Q10.G, Q18.C, Q19.G, R21.2, R42.2
- new net TO_BATT: C24.1, IC11.VIN, LED4.A, Q18.E, R22.2
- net GND: now also C15.-, C20.-, C21.1, C22.2, C23.1, C24.2, C26.2, C28.-, C31.1, D6.A, IC10.GND, IC11.GND, IC12.GND, IC12.VO, IC13.GND, IC15P.V-, IC8.GND, IC9.A, Q19.S, R15.2, R19.1, R28.2, R42.1, R45.2, R52.1
- net N$17: now also C20.+, IC8.VO, R16.2; no longer D5.A, IC8.SW, L2.2
- net N$19: now also IC8.EN, R47.2; no longer C20.1, IC8.FB, R15.1, R16.1
- net N$2: now also C21.2, IC8.ADJ, R15.1, R16.1; no longer C21.+, IC8.VIN, L2.1, R18.2
- net N$20: now also C15.+, C25.1, D7.C, IC8.VIN, Q17.S, R43.2, R47.1; no longer C15.-, C21.-, IC8.GND, R15.2
- net N$22: now also C23.2, IC11.VO; no longer IC9_3.3V2.OUT
- net N$23: now also D8.A, IC12.VIN, IC15P.V+, Q17.D, R48.2; no longer C15.+, C20.2, D5.C, R16.2
- net N$28: now also C29.2, D8.C, D9.A; no longer IC8.!SHDN!, R18.1
- net N$29: now also C26.1, IC10.VIN, L1.1, R44.2; no longer IC9_3.3V2.IN, LED4.A, Q18.E, R22.2
- net N$31: now also C25.2, IC10.FB, R28.1, R43.1; no longer IC9_3.3V2.ADJ
- net N$34: now also IC9.K; no longer IC9.C
- net N$36: now also C29.1, IC12.+CAP; no longer Q19.S
- net N$38: now also IC12.BOOST, IC15A.OUT, R48.1; no longer R42.1
Other:
- note added: "2Vin-2Vd= =12-[1.7(@-50C)..0.8(@125C)]= =10.3..11.2"
- note added: "3.5784 @1.278 3.472 @ typ 1.24 3.3656 @1.202 przy bledzie dzielnika 0.46% (rez. 1%)najwyzsze mozliwe napiecie to 3.595"
- note added: "R2 = R1 (Vout / 1.23 -1) R1=12k; R2=47k => Vout=6.05"
- note added: "Redundant voltage limiter - soft overvoltage protection with fault indicator"
- note added: "Vin ograniczony w zakresie Vcc-0.2 : Vee-1.1"
- note added: "Vo=1.242(1+R16/R15) & R45<470k for performance R15=10k; R16=33k => 5.00V"
- note added: "Vo=1.242(1+R45/R46) & R45<470k for performance R45=330k; R46=47k => 9.96V"
- note added: "sprawdz, czy rzeczywiscie dioda zaporowa dziala"
- note added: "voltage drop below 9.5 enables pump boost mode to compensate for eg. termal capacitance elements drop"
- note removed: "3.5784 @1.278 3.472 @ typ 1.24 3.3656 @1.202 przy bledzie dzielnika .46% (rez. 1%) najwyzsze mozliwe napiecie to 3.595"
- note removed: "R2 = R1 (Vout / 1.23 -1) R1=12k; R2=100k => Vout=11.48"
- moved on the sheet: C15, IC8, IC9, LED4, Q18, Q19, R15, R16, R18, R19, R20, R22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
