File: sensor-board2.sch (EAGLE design)
At the start: 154 parts, among them IC1 MCP3423, IC10 LM2731(X/Y), IC10_ADJ LD117AS12TR, IC11 TLV702, IC12 TC1044SEOA, IC13 MIC5209, IC15 LM393D, IC2 MPXHZ6115A6U, IC3 MPX2010, IC4 MAG3110, IC5 MMA8652FC, IC6 FXAS21002C, IC7 RFM95, IC8 MIC5209, IC8_5V LD117AS12TR, IC9 TLV431 (1.24VREF), IC9_3.3V LD117AS12TR, IC9_3.3V1 LD117AS12TR, J2 JP7, Q10 DMP3130L, Q17 DMP3130L, Q18 BC807-16LT1SMD, Q19 IRLML2060, X1 SMA-142-0701-801/806

Commit message: 12-10 care with the BOOST mode
Parts:
- added C27, C32: 1u/50V, rcl:C-EUC1206
- added D10, D5: 4001, diode:DIODE-DO-214AC
- added FDBK1: 680k, resistor:R-EU_R0805
- added IC14: TLV702, TI:TLV702
- added IC16: TLV431, TI:TL431-ASA
- added Q20: DMP3130L, miscrel:DMP3130L
- added R49: 390k, resistor:R-EU_R0805
- added R50: 12k, resistor:R-EU_R0805
- added R53: 22k, resistor:R-EU_R0805
- added R54: 39k, resistor:R-EU_R0805
- added R58: 68k, resistor:R-EU_R0805
- D6: value 3v3 -> 3V3
- R19, R29: value 100k -> 22k
- R20: value 180k -> 39k
- R21: value 1M -> 22k
- R22: value 1M -> 560k
- R48: value 1M -> 10k
- R51: value 100k -> 10k
- R52: value 15k -> 39k
Connections:
- removed net BOOST_SENS_A+: C31.2, IC13.ADJ, R45.1, R46.1
- removed net BOOST_SENS_A-: R51.1, R52.2
- removed net N$21: IC9.R, R19.2, R20.1
- new net BOOST_SENS_1.242: C31.2, IC13.ADJ, IC15A.+IN, R45.1, R46.1
- new net N$47: C27.2, IC14.VO, Q20.S
- new net N$48: IC14.EN
- new net N$49: Q20.D, R52.2
- new net N$50: FDBK1.1, IC9.R, R19.2, R20.1
- new net REF(1.24): IC16.K, IC16.R, R50.1, R51.1
- net GND: now also C27.1, C32.2, IC14.GND, IC16.A, R53.1, R58.2; no longer R52.1
- net N$17: now also D10.A
- net N$20: now also D10.C; no longer Q17.S
- net N$23: now also R50.2
- net N$38: now also R49.2
- net N$42: now also R52.1, R53.2; no longer IC15A.+IN
- net N$43: now also D5.C
- net N$44: now also D5.A; no longer R51.2
- net N$45: now also R49.1, R51.2, R58.1; no longer IC15A.-IN
- net REHREH: now also FDBK1.2
- net TO_BATT: now also C32.1, IC14.VIN
Other:
- note added: "0.61mA spoczynkowo 0.01mA + Iboost(0?) w stanie aktywnym"
- note added: "9.716*47/(47+330) = 1.2113 najnizsze mozliwe napiecie (sens.) wynikajace z odchylki dzielnika zadajacego (0,46%) i odchylki stabilizatora w dol: 2%V zadanego, przy którym wystąpi przelączenie powrotne komparatora dodatkowo nalezy odjac 11mV maksymalnego dryftu temperaturowego TLV431, co daje: 1.2003V przy gornej granicy histerezy w specyficznych, malo prawdopodobnych warunkach wystapi obszar zabl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"
- note added: "Ibias=100-10nA(max-typ) Vdrop=33mV-3.3mV"
- note added: "Napiecia REF z TLV431 REF -> Lo -> Hi 1.278 -> 1.098 -> 1.218 1.240 -> 1.057 -> 1.186 1.202 -> 1.025 -> 1.153"
- note added: "Napiecia SENS na MIC5209 REF -> Lo -> Hi 1.278 -> 8.807 -> 9.770 1.240 -> 8.479 -> 9.513 1.202 -> 8.221 -> 9.249"
- note added: "Vo=1.242(1+R45/R46) & R45<470k for performance R45=330k; R46=47k => 9.96V (typ.)"
- note added: "Vref=1.24"
- note added: "Vstab+/-2% (3.234-3.366)"
- note added: "Vstab+/-2% (9.76-10.16)"
- note added: "Wartosci napiec zabezpieczajacych: 3.618 @1.278 3.500 @ typ 1.24 3.400 @1.202 przy bledzie dzielnika 0.46% (rez. 1%) najwyzsze napiecie to 3.635 + 0.0195 najnizsze napiecie to 3.384"
- note added: "additional drop: 0.0195V Iref=0.5uA in worst case possile"
- note added: "ceramiczne kondensatory zwykle zawodzą zwierając - pakuj po dwa szeregowo"
- note added: "jesli TLV431 wpadnie w oscylacje, zmniejsz R22 do 100k puszczajac mu wiecej pradu"
- note added: "wejscia komparatora nie pobieraja pradu wiekszego niz 25nA, chyba ze zostanie podane na nie ujemne napiecie -0.3V"
- note added: "zadane napiecie: 9.96V moze dropnac do 99.54% z racji dzielnika nastepnie moze spacs do 97.55% przez +/-2% dryft temperaturowy w zakresie -55/+150 9.96 * 97.55% = 9.716V jest najnizszym napieciem stabilizowanym i jednoczsnie najwyzsza granica, ponizej ktorej nie wystapi BOOST latching."
- note removed: "3.5784 @1.278 3.472 @ typ 1.24 3.3656 @1.202 przy bledzie dzielnika 0.46% (rez. 1%)najwyzsze mozliwe napiecie to 3.595"
- note removed: "Vo=1.242(1+R45/R46) & R45<470k for performance R45=330k; R46=47k => 9.96V"
- note removed: "voltage drop below 9.5 enables pump boost mode to compensate for eg. termal capacitance elements drop"
- moved on the sheet: C15, C20, C21, C22, C25, C26, C28, C29, C30, C31, D7, D8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
