File: sensor-board2.sch (EAGLE design)
At the start: 167 parts, among them IC1 MCP3423, IC10 LM2731(X/Y), IC10_ADJ LD117AS12TR, IC11 TLV702, IC12 TC1044SEOA, IC13 MIC5209, IC14 TLV702, IC15 LM393D, IC16 TLV431, IC2 MPXHZ6115A6U, IC3 MPX2010, IC4 MAG3110, IC5 MMA8652FC, IC6 FXAS21002C, IC7 RFM95, IC8 MIC5209, IC8_5V LD117AS12TR, IC9 TLV431 (1.24VREF), IC9_3.3V LD117AS12TR, IC9_3.3V1 LD117AS12TR, J2 JP7, Q10 DMP3130L, Q17 DMP3130L, Q18 BC807-16LT1SMD, Q19 IRLML2060, Q20 DMP3130L, X1 SMA-142-0701-801/806

Commit message: All voltages protected
Parts:
- removed C30: 22u/25V, rcl:CPOL-EUC/6032-28R
- removed Q20: DMP3130L, miscrel:DMP3130L
- removed R52, R54: 39k, resistor:R-EU_R0805
- added D11, D12: 3V3, diode:ZENER-DIODESOD80C
- added FDBK2: 680k, resistor:R-EU_R0805
- added IC17: TLV431 (1.24VREF), TI:TL431-ASA
- added LED5: FAULT IND RED, eagle-ltspice:LED_E
- added Q21, Q24: DMP3130L, miscrel:DMP3130L
- added Q22: BC807-16LT1SMD, transistor-pnp:BC807-16LT1SMD
- added Q23: IRLML2060, miscrel:IRLML2060
- added R55, R57: 10k, resistor:R-EU_R0805
- added R56: 33k, resistor:R-EU_R0805
- added R59, R61, R64, R67: 22k, resistor:R-EU_R0805
- added R60: 910k, resistor:R-EU_R0805
- added R63: 560k, resistor:R-EU_R0805
- added R65: 3k3, resistor:R-EU_R0805
- added R66: 1k, resistor:R-EU_R0805
- R62: value 22k -> 39k
- renumbered R53 to R62
Connections:
- net POWER_FAULT_3V3_PLOGIC_CMOS renamed POWER_FAULT_3V3_LORA_PLOGIC_CMOS
- removed net N$42: R52.1, R62.2
- removed net N$47: C27.2, IC14.VO, Q20.S
- removed net N$49: Q20.D, R52.2
- new net 3V3_FOR_IMU: Q24.D, R62.2
- new net N$21: IC15B.OUT, Q21.G, R55.1, R59.1, R60.2
- new net N$51: Q21.D, R56.1
- new net N$52: Q22.B, R64.2
- new net N$53: IC17.K, R63.1, R64.1
- new net N$54: LED5.C, R66.1
- new net N$55: Q23.D, R66.2
- new net N$56: C27.2, IC14.VO, Q24.S
- new net N$57: FDBK2.1, IC17.R, R61.2, R62.1
- new net POWER_FAULT_3V3_IMU_CMOS_PLOGIC: D12.C, R67.1
- new net POWER_FAULT_5V_CPU_CMOS_PLOGIC: D11.C, R59.2
- new net REHREH1: FDBK2.2, Q22.C, Q23.G, Q24.G, R65.2, R67.2
- new net TO_BATT1: C32.1, IC14.VIN, LED5.A, Q22.E, R63.2
- net GND: now also D11.A, D12.A, IC17.A, Q23.S, R57.2, R61.1, R65.1; no longer R62.1
- net N$17: now also Q21.S, R55.2
- net N$29: now also IC15B.-IN, R56.2, R57.1, R60.1; no longer C26.1, IC10.VIN, L1.1, R44.2
- net REF(1.24): now also IC15B.+IN
- net TO_BATT: now also C26.1, IC10.VIN, L1.1, R44.2; no longer C32.1, IC14.VIN
Other:
- note added: "5.542 max_low (@1.278) hi 5.349 (no hist 5.495) 5.377 max_low (@1240) hi 5.190 (no hist 5.332) 5.212 max_low (@1.202) hi 5.03 (no hist 5.169) lo: 910||10 -d- 33 hi: (10+910)||33 -d- 10"
- note added: "Ibias=100-10nA(max-typ) Vdrop=10mV-1mV"
- note added: "Ibias=100-10nA(max-typ)++25nA z komparatora Vdrop=33mV-3.3mV++8.25mV"
- note added: "Napiecie wyjsciowe moze sie podniesc o 2% od napiecia zadanego na skutek temperatury, a nastepnie o 0.46% przez blad dzielnika. Finalnie 100.46%*102%=102.47% Vmax=5.12 (+40mV z Ibias) - powyzej tego zabezpieczac (REF>5.106*(33/100)-10mV=1.257)"
- note added: "POWER_OK zrob bramka AND"
- note added: "Vo=1.242(1+R16/R15) & R_upper<470k for performance Rup=100k; Rdwn=33k => 5.006V +/-2% +/-0.46% 4.905 - 5.006(nom) - 5.106"
- note added: "Vo=1.242(1+R45/R46) & R_upper<470k for performance Rup=330k; Rdwn=47k => 9.96V (typ.)"
- note added: "Vstab +/-2% +/-0.46% 9.72 - 9.96(nom) - 10.21"
- note added: "Wartosci napiec zabezpieczajacych: Lo: 3.618 @1.278 HI: 3.413(3V5); 3.374(4V2) Lo: 3.500 @ typ 1.24 HI: 3.307(3V5); 3.272(4V2) Lo: 3.400 @1.202 HI: 3.200(3V5) ;3.162(4V2) przy bledzie dzielnika 0.46% (rez. 1%) najwyzsze napiecie to 3.635 + 0.0195 najnizsze napiecie to 3.384"
- note added: "Zredukuj wartosci rezystorow dla zwiekszenia precyzji nastaw napiec"
- note added: "górne zabezpieczenie max.5.5V (REF=5.5*(33/133)-12.5mV=1.352V) REF*99.54%=1.346V"
- note added: "zadane napiecie: 9.96V moze dropnac do 99.54% z racji dzielnika nastepnie moze spacs do 97.55% przez +/-2% dryft temperaturowy w zakresie -55/+150 9.96 * 97.55% (-330mV z Ibias) = 9.718V jest najnizszym napieciem stabilizowanym i jednoczesnie powinno być wzięte za najwyzsza granice, ponizej ktorej nie wystapi BOOST latching. Ibias nie wliczano i moze spowodowac dalsze ryzyko BOOST latching (zazna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"
- note removed: "Ibias=100-10nA(max-typ) Vdrop=33mV-3.3mV"
- note removed: "Vo=1.242(1+R16/R15) & R45<470k for performance R15=10k; R16=33k => 5.00V"
- note removed: "Vo=1.242(1+R45/R46) & R45<470k for performance R45=330k; R46=47k => 9.96V (typ.)"
- note removed: "Vstab+/-2% (9.76-10.16)"
- note removed: "Wartosci napiec zabezpieczajacych: 3.618 @1.278 3.500 @ typ 1.24 3.400 @1.202 przy bledzie dzielnika 0.46% (rez. 1%) najwyzsze napiecie to 3.635 + 0.0195 najnizsze napiecie to 3.384"
- note removed: "zadane napiecie: 9.96V moze dropnac do 99.54% z racji dzielnika nastepnie moze spacs do 97.55% przez +/-2% dryft temperaturowy w zakresie -55/+150 9.96 * 97.55% = 9.716V jest najnizszym napieciem stabilizowanym i jednoczsnie najwyzsza granica, ponizej ktorej nie wystapi BOOST latching."
- moved on the sheet: C20, C22, C27, C32, IC14, IC15B

Commit message: Project leakage revoked
All retards cured witch charger schem.
Parts:
- removed C21, C31: 470p/50V, rcl:C-EUC1206
- removed C32: 1u/50V, rcl:C-EUC1206
- added C30: 1n/50V, rcl:C-EUC1206
- added C33, C34, C35, C36: 4u7/16V, resistor:CPOL-EUSMCB
- added D13, D14, D15: 3V3, diode:ZENER-DIODESOD80C
- added IC18: MCP73871, TI:MCP73871
- added R52: 10k NTC B=3950, ptc-ntc:NTC640-9
- added R53: 2k2, resistor:R-EU_R0805
- added R54: 68k, resistor:R-EU_R0805
- added R68, R72: 100k, resistor:R-EU_R0805
- added R69: 33k, resistor:R-EU_R0805
- added R70, R71: 680k, resistor:R-EU_R0805
- added R73: 910k, resistor:R-EU_R0805
- added R74, R75, R76: 10k, resistor:R-EU_R0805
- added T1: IRLML2060, miscrel:IRLML2060
- C25: value 560p/50V -> 1n/50V
- C26: value 4u7/16V -> 10u/16V
- R18, R44, R47: value 56k -> 680k
Connections:
- net N$44 renamed PWR_FOR_PRESS
- net N$51 renamed 5V_FOR_ESP32_&_AUXADC
- removed net LOW_SHDN_6V: IC10.!SHDN!, R44.1
- removed net PUMP_HI_TO_SHDN: Q17.G
- new net BOOST_BATT: C26.1, IC10.VIN, L1.1, R44.2
- new net LOW-USB(100MA)/HIGH-ADAPTER(1.8A): IC18.SEL
- new net N$42: R52.2, R53.1, R54.2
- new net N$44: D15.C, R74.2
- new net N$47: IC18.THERM, R53.2
- new net N$49: C34.+, IC18.VOUT
- new net N$58: C35.+, IC18.VBAT
- new net N$59: C36.+, IC18.VIN, R68.2
- new net N$60: IC18.VPCC, R68.1, R69.1
- new net N$61: D14.C, R76.1
- new net N$62: C25.1, C30.2
- new net PWR_BOOST_!SHDN!: IC10.!SHDN!, R44.1, R74.1
- new net PWR_IMU_!SHDN!: IC14.EN, R71.2, R76.2
- new net PWR_LORA_!SHDN!: IC11.EN, R70.2, R75.2
- new net PWR_PRESS_!SHDN!: R73.1, T1.G
- net BOOST_SENS_1.242: no longer C31.2
- net GND: now also C23.2, C34.-, C35.-, C36.-, D13.A, D14.A, D15.A, IC18.VSS, R52.1, R54.1, R69.2, T1.S; no longer C21.1, C23.1, C31.1, C32.2
- net N$2: no longer C21.2
- net N$20: now also C30.1, Q17.S, R72.2, R73.2; no longer C25.1
- net N$22: now also C23.1; no longer C23.2
- net N$26: now also Q17.G, R72.1, T1.D; no longer IC11.EN
- net N$48: now also D13.C, R75.1; no longer IC14.EN
- net TO_BATT: now also R70.1; no longer C26.1, IC10.VIN, L1.1, R44.2
- net TO_BATT1: now also R71.1; no longer C32.1
Other:
- note added: "9.716*47/(47+330) = 1.214 najnizsze mozliwe napiecie (sens.) wynikajace z odchylki dzielnika zadajacego (0.22%) i odchylki stabilizatora w dol: 2%V zadanego, przy ktorym wystapi przelaczenie powrotne omparatora W specyficznych, malo prawdopod. warunkach wystapi obszar zablokowania komparatora w pozycji BOOST_ON (9.74 SENS. nie bedzie w stanie przekroczyc wymaganych 9.77) efektem spadek efektywnos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"
- note added: "Cel: nie dopuszczac napiecia powyzej 5.5V Obszary dzialania histerezy: (@1.278) 5.542-low_hi -> 5.349-high_hi (no hist-5.495) (@1.240) 5.377-low_hi -> 5.190-high_hi (no hist 5.332) (@1.202) 5.212-low_hi -> 5.030-high_hi (no hist 5.169) dzielnik do liczenia histerezy: lo: 910||10 -d- 33 hi: (10+910)||33 -d- 10"
- note added: "Granice temperatur ladowania: Th=46.6C Tl=0.88C"
- note added: "Ibias=100-10nA(max-typ)++25nA z komparatora Vdrop=33mV..3.3mV++8.25mV"
- note added: "Napiecia SENS na MIC5209 i wynikajace z nich napiecia linii 10V zal / wyl komparator i BOOST REF -> Lo -> Hi 1.278 -> 8.807 -> 9.770 1.240 -> 8.479 -> 9.513 1.202 -> 8.221 -> 9.249"
- note added: "Napiecie wyjsciowe moze sie podniesc o 2% od napiecia zadanego na skutek temperatury, a nastepnie o 0.37% przez blad dzielnika. Finalnie 100.37%*102%=102.38% Vmax=5.125 (+40mV z Ibias po przekladni dzielnika) - - obszar napiec zabezpieczajacych powinien byc powyzej"
- note added: "UVLO - wylacza Vout, poki napiecie nie przekroczy 1.9V"
- note added: "Uwaga! Wyjscie tylko do obserwacji! Nie sterowac go!"
- note added: "VPCC shuts down charging in favor of powered circuit in case of input power shortage Vtrigger=1.23V Vlow=4.96"
- note added: "Vo=1.242(1+R16/R15) & R_upper<470k for performance Rup=100k; Rdwn=33k => 5.006V +/-2% +/-0.37% 4.928 - 5.006(nom) - 5.165"
- note added: "Vo=1.242(1+Rup/Rdwn) & R_upper<470k for performance Rup=330k; Rdwn=47k => 9.96V (typ.)"
- note added: "Vstab +/-2% +/-0.22% 9.74 - 9.96(nom) - 10.18 vdrop * (377/47)=+(93..330)mV"
- note added: "dla zmniejszenia rozrzutu nastaw napiec zredukowac wartosci resystorow"
- note added: "zadane napiecie: 9.96V moze dropnac do 99.78% z racji dzielnika nastepnie moze spacs do 97.78% przez +/-2% dryft temperaturowy w zakresie -55/+150 9.96 * 97.78% = 9.740V jest najnizszym napieciem stabilizowanym i jednoczesnie powinno byc wziete za najwyzsza granice, ponizej ktorej nie wystapi BOOST latching."
- note removed: "5.542 max_low (@1.278) hi 5.349 (no hist 5.495) 5.377 max_low (@1240) hi 5.190 (no hist 5.332) 5.212 max_low (@1.202) hi 5.03 (no hist 5.169) lo: 910||10 -d- 33 hi: (10+910)||33 -d- 10"
- note removed: "9.716*47/(47+330) = 1.2113 najnizsze mozliwe napiecie (sens.) wynikajace z odchylki dzielnika zadajacego (0,46%) i odchylki stabilizatora w dol: 2%V zadanego, przy którym wystąpi przelączenie powrotne komparatora dodatkowo nalezy odjac 11mV maksymalnego dryftu temperaturowego TLV431, co daje: 1.2003V przy gornej granicy histerezy w specyficznych, malo prawdopodobnych warunkach wystapi obszar zabl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"
- note removed: "Ibias=100-10nA(max-typ)++25nA z komparatora Vdrop=33mV-3.3mV++8.25mV"
- note removed: "Napiecia SENS na MIC5209 REF -> Lo -> Hi 1.278 -> 8.807 -> 9.770 1.240 -> 8.479 -> 9.513 1.202 -> 8.221 -> 9.249"
- note removed: "Napiecie wyjsciowe moze sie podniesc o 2% od napiecia zadanego na skutek temperatury, a nastepnie o 0.46% przez blad dzielnika. Finalnie 100.46%*102%=102.47% Vmax=5.12 (+40mV z Ibias) - powyzej tego zabezpieczac (REF>5.106*(33/100)-10mV=1.257)"
- note removed: "POWER_OK zrob bramka AND"
- note removed: "Vo=1.242(1+R16/R15) & R_upper<470k for performance Rup=100k; Rdwn=33k => 5.006V +/-2% +/-0.46% 4.905 - 5.006(nom) - 5.106"
- note removed: "Vo=1.242(1+R45/R46) & R_upper<470k for performance Rup=330k; Rdwn=47k => 9.96V (typ.)"
- note removed: "Vref=1.24"
- note removed: "Vstab +/-2% +/-0.46% 9.72 - 9.96(nom) - 10.21"
- note removed: "Zredukuj wartosci rezystorow dla zwiekszenia precyzji nastaw napiec"
- note removed: "ceramiczne kondensatory zwykle zawodzą zwierając - pakuj po dwa szeregowo"
- note removed: "górne zabezpieczenie max.5.5V (REF=5.5*(33/133)-12.5mV=1.352V) REF*99.54%=1.346V"
- note removed: "zadane napiecie: 9.96V moze dropnac do 99.54% z racji dzielnika nastepnie moze spacs do 97.55% przez +/-2% dryft temperaturowy w zakresie -55/+150 9.96 * 97.55% (-330mV z Ibias) = 9.718V jest najnizszym napieciem stabilizowanym i jednoczesnie powinno być wzięte za najwyzsza granice, ponizej ktorej nie wystapi BOOST latching. Ibias nie wliczano i moze spowodowac dalsze ryzyko BOOST latching (zazna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"
- moved on the sheet: C15, C20, C23, C24, C25, C26, C27, D12, D6, D7, FDBK1, FDBK2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

Commit message: file cleaning
Changed lines of the file:
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@@
 <part name="R76" library="resistor" deviceset="R-EU_" device="R0805" value="10k"/>
 <part name="C30" library="rcl" deviceset="C-EU" device="C1206" value="1n/50V"/>
+<part name="GND48" library="supply1" deviceset="GND" device=""/>
 </parts>
 <sheets>
@@
 <instance part="IC14" gate="G$1" x="-391.16" y="-396.24"/>
 <instance part="C27" gate="G$1" x="-375.92" y="-408.94" rot="R180"/>
-<instance part="GND59" gate="1" x="-391.16" y="-434.34"/>
+<instance part="GND59" gate="1" x="-391.16" y="-426.72"/>
 <instance part="FDBK1" gate="G$1" x="-302.26" y="-314.96" rot="R180"/>
 <instance part="D5" gate="G$1" x="-391.16" y="-198.12" rot="MR0"/>
@@
 <instance part="GND78" gate="1" x="-411.48" y="-340.36"/>
 <instance part="D13" gate="G$1" x="-401.32" y="-325.12" rot="R90"/>
-<instance part="GND79" gate="1" x="-401.32" y="-332.74"/>
+<instance part="GND79" gate="1" x="-401.32" y="-340.36"/>
 <instance part="T1" gate="G$1" x="-444.5" y="-182.88" rot="MR0"/>
 <instance part="R72" gate="G$1" x="-444.5" y="-160.02" rot="R90"/>
@@
 <instance part="R76" gate="G$1" x="-401.32" y="-408.94" rot="R90"/>
 <instance part="C30" gate="G$1" x="-497.84" y="-162.56" rot="R270"/>
+<instance part="GND48" gate="1" x="-375.92" y="-426.72"/>
 </instances>
 <busses>
@@
 <segment>
 <pinref part="IC14" gate="G$1" pin="GND"/>
-<wire x1="-391.16" y1="-421.64" x2="-391.16" y2="-403.86" width="0.1524" layer="91"/>
-<wire x1="-375.92" y1="-421.64" x2="-391.16" y2="-421.64" width="0.1524" layer="91"/>
-<junction x="-391.16" y="-421.64"/>
+<wire x1="-391.16" y1="-424.18" x2="-391.16" y2="-403.86" width="0.1524" layer="91"/>
 <pinref part="GND59" gate="1" pin="GND"/>
-<wire x1="-391.16" y1="-421.64" x2="-391.16" y2="-431.8" width="0.1524" layer="91"/>
-<pinref part="C27" gate="G$1" pin="1"/>
-<wire x1="-375.92" y1="-411.48" x2="-375.92" y2="-421.64" width="0.1524" layer="91"/>
 </segment>
 <segment>
@@
 <pinref part="D13" gate="G$1" pin="A"/>
 <pinref part="GND79" gate="1" pin="GND"/>
-<wire x1="-401.32" y1="-330.2" x2="-401.32" y2="-327.66" width="0.1524" layer="91"/>
+<wire x1="-401.32" y1="-337.82" x2="-401.32" y2="-327.66" width="0.1524" layer="91"/>
 </segment>
 <segment>
@@
 <wire x1="-543.56" y1="-177.8" x2="-543.56" y2="-180.34" width="0.1524" layer="91"/>
 </segment>
+<segment>
+<pinref part="C27" gate="G$1" pin="1"/>
+<wire x1="-375.92" y1="-411.48" x2="-375.92" y2="-424.18" width="0.1524" layer="91"/>
+<pinref part="GND48" gate="1" pin="GND"/>
+</segment>
 </net>
