File: sensor-board2.brd (EAGLE design)
At the start: 183 parts, among them IC1 MCP3423, IC10 LM2731(X/Y), IC10_ADJ LD117AS12TR, IC11 TLV702, IC12 TC1044SEOA, IC13 MIC5209, IC14 TLV702, IC15 LM393D, IC16 TLV431, IC17 TLV431 (1.24VREF), IC2 MPXHZ6115A6U, IC3 MPX2010, IC4 MAG3110, IC5 MMA8652FC, IC6 FXAS21002C, IC7 RFM95, IC8 MIC5209, IC8_5V LD117AS12TR, IC9 TLV431 (1.24VREF), IC9_3.3V LD117AS12TR, IC9_3.3V1 LD117AS12TR, J2 JP7, Q10 DMP3130L, Q17 DMP3130L, Q18 BC807-16LT1SMD, Q19 IRLML2060, Q21 DMP3130L, Q22 BC807-16LT1SMD, Q23 IRLML2060, Q24 DMP3130L, X1 SMA-142-0701-801/806

Commit message: Project leakage revoked
All retards cured witch charger schem.
Parts:
- removed C21, C31: 470p/50V, rcl:C1206
- removed C32: 1u/50V, rcl:C1206
- added C30: 1n/50V, rcl:C1206
- added C33, C34, C35, C36: 4u7/16V, resistor:SMC_B
- added D13, D14, D15: 3V3, diode:SOD80C
- added IC18: MCP73871, TI:QFN-20
- added R52: 10k NTC B=3950, ptc-ntc:N640
- added R53: 2k2, resistor:R0805
- added R54: 68k, resistor:R0805
- added R68, R72: 100k, resistor:R0805
- added R69: 33k, resistor:R0805
- added R70, R71: 680k, resistor:R0805
- added R73: 910k, resistor:R0805
- added R74, R75, R76: 10k, resistor:R0805
- added T1: IRLML2060, miscrel:SOT23-3
- C25: value 560p/50V -> 1n/50V
- C26: value 4u7/16V -> 10u/16V
- R18, R44, R47: value 56k -> 680k
Connections:
- net N$44 renamed PWR_FOR_PRESS
- net N$51 renamed 5V_FOR_ESP32_&_AUXADC
- removed net LOW_SHDN_6V: IC10.4, R44.1
- removed net PUMP_HI_TO_SHDN: Q17.1
- new net !PG!: IC18.6
- new net BOOST_BATT: C26.1, IC10.5, L1.1, R44.2
- new net LOW-USB(100MA)/HIGH-ADAPTER(1.8A): IC18.3
- new net N$42: R52.2, R53.1, R54.2
- new net N$44: D15.C, R74.2
- new net N$47: IC18.5, R53.2
- new net N$49: C34.+, IC18.1, IC18.20
- new net N$58: C35.+, IC18.14, IC18.15, IC18.16
- new net N$59: C36.+, IC18.18, IC18.19, R68.2
- new net N$60: IC18.2, R68.1, R69.1
- new net N$61: D14.C, R76.1
- new net N$62: C25.1, C30.2
- new net PWR_BOOST_!SHDN!: IC10.4, R44.1, R74.1
- new net PWR_IMU_!SHDN!: IC14.3, R71.2, R76.2
- new net PWR_LORA_!SHDN!: IC11.3, R70.2, R75.2
- new net PWR_PRESS_!SHDN!: R73.1, T1.1
- net BOOST_SENS_1.242: no longer C31.2
- net GND: now also C23.2, C34.-, C35.-, C36.-, D13.A, D14.A, D15.A, IC18.10, IC18.11, IC18.EXP, R52.1, R54.1, R69.2, T1.2; no longer C21.1, C23.1, C31.1, C32.2
- net N$2: no longer C21.2
- net N$20: now also C30.1, Q17.2, R72.2, R73.2; no longer C25.1
- net N$22: now also C23.1; no longer C23.2
- net N$26: now also Q17.1, R72.1, T1.3; no longer IC11.3
- net N$48: now also D13.C, R75.1; no longer IC14.3
- net TO_BATT: now also R70.1; no longer C26.1, IC10.5, L1.1, R44.2
- net TO_BATT1: now also R71.1; no longer C32.1
